Commit message: Updated robot model, URDF, and design files (clean sync)

File: hardware/fyp_robot_urdf/urdf/fyp_robot_urdf.urdf (robot description, URDF)
Before this commit: robot fyp_robot_assem, 3 links, 2 joints
Links:
- link base_link: geometry collision mesh filename=package://fyp_robot_urdf/meshes/base_link.STL; visual mesh filename=package://fyp_robot_urdf/meshes/base_link.STL
- link link1: mass 0.234233661750754 -> 0.234233603955478; geometry collision mesh filename=package://fyp_robot_urdf/meshes/link1.STL; visual mesh filename=package://fyp_robot_urdf/meshes/link1.STL
- link link2: mass 0.175905996218137 -> 0.175905723230877; geometry collision mesh filename=package://fyp_robot_urdf/meshes/link2.STL; visual mesh filename=package://fyp_robot_urdf/meshes/link2.STL
Joints:
- joint joint1: axis 0 0 1 -> 0 0 -1; limit (none) -> lower=-1.5708 upper=1.5708 effort=8 velocity=30; origin xyz=0.0175 0 0.0373735903262573 rpy=-1.5707963267949 0 -1.5707963267949 -> xyz=0.0175 0 0.03735 rpy=-1.5708 0 -1.5708; type continuous -> revolute
- joint joint2: axis 0 0 1 -> 0 0 -1; limit (none) -> lower=-1.5708 upper=1.5708 effort=8 velocity=30; origin xyz=-0.156657030121427 -0.194776017515082 0.0425 rpy=0 0 0 -> xyz=0 -0.25 0.0425 rpy=0 0 0; type continuous -> revolute
